Commit message: split into proper urdf structure

File: ros2/description/urdf/tibble.urdf.xacro (robot description, xacro)
@@ -1,990 +1,17 @@
 <?xml version="1.0" encoding="utf-8"?>
-<!-- This URDF was automatically created by SolidWorks to URDF Exporter! Originally created by Stephen Brawner (brawner@gmail.com)
-     Commit Version: 1.6.0-4-g7f85cfe  Build Version: 1.6.7995.38578
-     For more information, please see http://wiki.ros.org/sw_urdf_exporter -->
-<robot
-  name="tibble">
-  <link name="base_link"/>
-  <link
-    name="chassis_link">
-    <inertial>
-      <origin
-        xyz="0.88193 1.2843 1.595"
-        rpy="0 0 0" />
-      <mass
-        value="5.3252" />
-      <inertia
-        ixx="0.016501"
-        ixy="-1.6464E-09"
-        ixz="0.0014196"
-        iyy="0.28053"
-        iyz="3.4252E-11"
-        izz="0.27372" />
-    </inertial>
-    <visual>
-      <origin
-        xyz="0 0 0"
-        rpy="0 0 0" />
-      <geometry>
-        <mesh
-          filename="file://$(find description)/meshes/Chassis.STL" />
-      </geometry>
-      <material
-        name="">
-        <color
-          rgba="0.25098 0.25098 0.25098 1" />
-      </material>
-    </visual>
-    <collision>
-      <origin
-        xyz="0 0 0"
-        rpy="0 0 0" />
-      <geometry>
-        <mesh
-          filename="file://$(find description)/meshes/Chassis.STL" />
-      </geometry>
-    </collision>
-  </link>
-  <joint
-    name="chassis"
-    type="fixed">
-    <origin
-      xyz="0 0 0"
-      rpy="${-pi/2} 0 0" />
-    <parent
-      link="base_link" />
-    <child
-      link="chassis_link" />
-  </joint>
-  <link
-    name="DL_Wheel">
-    <inertial>
-      <origin
-        xyz="-2.6735E-11 -2.2271E-11 5.6577E-12"
-        rpy="0 0 0" />
-      <mass
-        value="0.17677" />
-      <inertia
-        ixx="0.00011937"
-        ixy="-6.5392E-14"
-        ixz="3.4896E-14"
-        iyy="0.00011937"
-        iyz="-1.0101E-14"
-        izz="0.00021546" />
-    </inertial>
-    <visual>
-      <origin
-        xyz="0 0 0"
-        rpy="0 0 0" />
-      <geometry>
-        <mesh
-          filename="file://$(find description)/meshes/DL_Wheel.STL" />
-      </geometry>
-      <material
-        name="">
-        <color
-          rgba="0.79216 0.81961 0.93333 1" />
-      </material>
-    </visual>
-    <collision>
-      <origin
-        xyz="0 0 0"
-        rpy="0 0 0" />
-      <geometry>
-        <mesh
-          filename="file://$(find description)/meshes/DL_Wheel.STL" />
-      </geometry>
-    </collision>
-  </link>
-  <joint
-    name="DL_Rotate"
-    type="continuous">
-    <origin
-      xyz="1.1775 -1.6339 1.5673"
-      rpy="3.1416 0 0.5236" />
-    <parent
-      link="chassis_link" />
-    <child
-      link="DL_Wheel" />
-    <axis
-      xyz="0 0 -1" />
-  </joint>
-  <link
-    name="DR_Wheel">
-    <inertial>
-      <origin
-        xyz="-2.67351696336959E-11 -2.22715179631905E-11 5.65791857809472E-12"
-        rpy="0 0 0" />
-      <mass
-        value="0.176769243894823" />
-      <inertia
-        ixx="0.000119374362744726"
-        ixy="-6.53920243420727E-14"
-        ixz="3.48950358018505E-14"
-        iyy="0.000119374363023012"
-        iyz="-1.01023471885648E-14"
-        izz="0.000215461530204446" />
-    </inertial>
-    <visual>
-      <origin
-        xyz="0 0 0"
-        rpy="0 0 0" />
-      <geometry>
-        <mesh
-          filename="file://$(find description)/meshes/DR_Wheel.STL" />
-      </geometry>
-      <material
-        name="">
-        <color
-          rgba="0.792156862745098 0.819607843137255 0.933333333333333 1" />
-      </material>
-    </visual>
-    <collision>
-      <origin
-        xyz="0 0 0"
-        rpy="0 0 0" />
-      <geometry>
-        <mesh
-          filename="file://$(find description)/meshes/DR_Wheel.STL" />
-      </geometry>
-    </collision>
-  </link>
-  <joint
-    name="DR_Rotate"
-    type="continuous">
-    <origin
-      xyz="1.1775 -1.6339 1.0014"
-      rpy="3.1416 0 0.5236" />
-    <parent
-      link="chassis_link" />
-    <child
-      link="DR_Wheel" />
-    <axis
-      xyz="0 0 -1" />
-  </joint>
-  <link
-    name="BLA">
-    <inertial>
-      <origin
-        xyz="-0.0172681243630312 -0.116440645758096 0.212737229814056"
-        rpy="0 0 0" />
-      <mass
-        value="0.97023402841067" />
-      <inertia
-        ixx="0.00819569952353813"
-        ixy="0.000828153171744282"
-        ixz="-1.42662335730119E-06"
-        iyy="0.000699830914870433"
-        iyz="3.45710523187761E-06"
-        izz="0.00867844294735175" />
-    </inertial>
-    <visual>
-      <origin
-        xyz="0 0 0"
-        rpy="0 0 0" />
-      <geometry>
-        <mesh
-          filename="file://$(find description)/meshes/BLA.STL" />
-      </geometry>
-      <material
-        name="">
-        <color
-          rgba="0.792156862745098 0.819607843137255 0.933333333333333 1" />
-      </material>
-    </visual>
-    <collision>
-      <origin
-        xyz="0 0 0"
-        rpy="0 0 0" />
-      <geometry>
-        <mesh
-          filename="file://$(find description)/meshes/BLA.STL" />
-      </geometry>
-    </collision>
-  </link>
-  <joint
-    name="LLA_Rotate"
-    type="revolute">
-    <origin
-      xyz="0.56252 -1.6364 1.0715"
-      rpy="0 0 0.88895" />
-    <parent
-      link="chassis_link" />
-    <child
-      link="BLA" />
-    <axis
-      xyz="0 0 -1" />
-    <limit
-      lower="0"
-      upper="0"
-      effort="0"
-      velocity="0" />
-  </joint>
-  <link
-    name="LA">
-    <inertial>
-      <origin
-        xyz="0.0420523159099391 0.0218514549059925 3.83189571184772E-08"
-        rpy="0 0 0" />
-      <mass
-        value="0.0898377249563414" />
-      <inertia
-        ixx="0.000634301272313686"
-        ixy="-3.23718441672287E-11"
-        ixz="-1.23742704912369E-10"
-        iyy="4.44119295047458E-06"
-        iyz="1.42114602862497E-10"
-        izz="0.000634330189167566" />
-    </inertial>
-    <visual>
-      <origin
-        xyz="0 0 0"
-        rpy="0 0 0" />
-      <geometry>
-        <mesh
-          filename="file://$(find description)/meshes/LA.STL" />
-      </geometry>
-      <material
-        name="">
-        <color
-          rgba="0.792156862745098 0.819607843137255 0.933333333333333 1" />
-      </material>
-    </visual>
-    <collision>
-      <origin
-        xyz="0 0 0"
-        rpy="0 0 0" />
-      <geometry>
-        <mesh
-          filename="file://$(find description)/meshes/LA.STL" />
-      </geometry>
-    </collision>
-  </link>
-  <joint
-    name="LA_Extend"
-    type="prismatic">
-    <origin
-      xyz="0.042052 -0.26173 0.40387"
-      rpy="-3.1416 0 3.1416" />
-    <parent
-      link="BLA" />
-    <child
-      link="LA" />
-    <axis
-      xyz="0 1 0" />
-    <limit
-      lower="0"
-      upper="0"
-      effort="0"
-      velocity="0" />
-  </joint>
-  <link
-    name="TLA">
-    <inertial>
-      <origin
-        xyz="0.042052315909939 0.0118514549059932 3.83189571184772E-08"
-        rpy="0 0 0" />
-      <mass
-        value="0.0898377249563407" />
-      <inertia
-        ixx="0.00063430127231368"
-        ixy="-3.23718437638293E-11"
-        ixz="-1.23742704915399E-10"
-        iyy="4.44119295047454E-06"
-        iyz="1.42114603355188E-10"
-        izz="0.00063433018916756" />
-    </inertial>
-    <visual>
-      <origin
-        xyz="0 0 0"
-        rpy="0 0 0" />
-      <geometry>
-        <mesh
-          filename="file://$(find description)/meshes/TLA.STL" />
-      </geometry>
-      <material
-        name="">
-        <color
-          rgba="0.792156862745098 0.819607843137255 0.933333333333333 1" />
-      </material>
-    </visual>
-    <collision>
-      <origin
-        xyz="0 0 0"
-        rpy="0 0 0" />
-      <geometry>
-        <mesh
-          filename="file://$(find description)/meshes/TLA.STL" />
-      </geometry>
-    </collision>
-  </link>
-  <joint
-    name="TLA_Rotate"
-    type="revolute">
-    <origin
-      xyz="0 0.01 0"
-      rpy="0 0 0" />
-    <parent
-      link="LA" />
-    <child
-      link="TLA" />
-    <axis
-      xyz="0 0 1" />
-    <limit
-      lower="0"
-      upper="0"
-      effort="0"
-      velocity="0" />
-  </joint>
-  <link
-    name="Hopper">
-    <inertial>
-      <origin
-        xyz="-0.218032737839366 -0.048578033407676 0.255785650299991"
-        rpy="0 0 0" />
-      <mass
-        value="7.0102265846381" />
-      <inertia
-        ixx="0.239055753793241"
-        ixy="-3.42031876735411E-05"
-        ixz="-5.68944981457304E-05"
-        iyy="0.257861535313843"
-        iyz="-0.00276345589773509"
-        izz="0.186808546830502" />
-    </inertial>
-    <visual>
-      <origin
-        xyz="0 0 0"
-        rpy="0 0 0" />
-      <geometry>
-        <mesh
-          filename="file://$(find description)/meshes/Hopper.STL" />
-      </geometry>
-      <material
-        name="">
-        <color
-          rgba="0.866666666666667 0.909803921568627 1 1" />
-      </material>
-    </visual>
-    <collision>
-      <origin
-        xyz="0 0 0"
-        rpy="0 0 0" />
-      <geometry>
-        <mesh
-          filename="file://$(find description)/meshes/Hopper.STL" />
-      </geometry>
-    </collision>
-  </link>
-  <joint
-    name="Hopper_Rotate"
-    type="revolute">
-    <origin
-      xyz="0.37173 -1.5824 1.0636"
-      rpy="0.03431 1.5708 0" />
-    <parent
-      link="chassis_link" />
-    <child
-      link="Hopper" />
-    <axis
-      xyz="1 0 0" />
-    <limit
-      lower="0"
-      upper="0"
-      effort="0"
-      velocity="0" />
-  </joint>
-  <link
-    name="Hopper_Door">
-    <inertial>
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