Commit message: added in new urdf but it is identical to the old one

File: ros2/description/urdf/tibble_core_old.xacro (robot description, xacro)
@@ -44,5 +44,5 @@
     </collision>
   </link>
-    <joint
+  <joint
     name="chassis"
     type="fixed">
@@ -275,5 +275,5 @@
       upper="0.254"
       effort="2000"
-      velocity="0.006" />
+      velocity="0.006" /> <!-- upper: 10 inch stroke. effort: 250lbs max load into newtons. velocity: 6mm/s into m/s -->
   </joint>
   <link
@@ -389,5 +389,5 @@
     <limit
       lower="-1"
-      upper="0"
+      upper="1"
       effort="0"
       velocity="0" />
