Commit message: Added basic gazebo references to the links

File: ros2/description/urdf/gazebo.xacro (robot description, xacro)
@@ -9,4 +9,129 @@
         <mu1 value="0.0"/>  <!-- This is friction -->
         <mu2 value="0.0"/>
+    </gazebo>
+    <gazebo reference="DL_Wheel">
+        <material>
+            <color rgba="0.79216 0.81961 0.93333 1" />
+        </material>
+        <!-- Arbitrary friction values -->
+        <mu1 value="0.001"/>
+        <mu2 value="0.001"/>
+    </gazebo>
+    <gazebo reference="DR_Wheel">
+        <material>
+            <color rgba="0.792156862745098 0.819607843137255 0.933333333333333 1" />
+        </material>
+        <!-- Arbitrary friction values -->
+        <mu1 value="0.001"/>
+        <mu2 value="0.001"/>
+    </gazebo>
+    <gazebo reference="BLA">
+        <material>
+            <color rgba="0.792156862745098 0.819607843137255 0.933333333333333 1" />
+        </material>
+        <!-- TODO: Any other configurations for Linear Actuators -->
+    </gazebo>
+    <gazebo reference="LA">
+        <material>
+            <color rgba="0.792156862745098 0.819607843137255 0.933333333333333 1" />
+        </material>
+        <!-- TODO: Any other configurations for Linear Actuators -->
+    </gazebo>
+    <!-- Not sure if this is a wheel or a linear actuator -->
+    <gazebo reference="TLA">
+        <material>
+            <color rgba="0.792156862745098 0.819607843137255 0.933333333333333 1" />
+        </material>
+        <!-- Included in case its a wheel -->
+        <mu1 value="0.001"/>
+        <mu2 value="0.001"/>
+    </gazebo>
+    <gazebo reference="Hopper">
+        <material>
+            <color rgba="0.866666666666667 0.909803921568627 1 1" />
+        </material>
+        <!-- TODO: Any other configurations for the Hopper -->
+    </gazebo>
+    <gazebo reference="Hopper_Door">
+        <material>
+            <color rgba="0.866666666666667 0.909803921568627 1 1" />
+        </material>
+        <!-- TODO: Any other configurations for the Hopper Door -->
+    </gazebo>
+    <gazebo reference="Hopper_Latch">
+        <material>
+            <color rgba="1 0 1 1" />
+        </material>
+        <!-- TODO: Any other configurations for the Hopper Latch -->
+    </gazebo>
+    <gazebo reference="Excavation">
+        <material>
+            <color rgba="0.792156862745098 0.819607843137255 0.933333333333333 1" />
+        </material>
+        <!-- TODO: Any other configurations for Excavation -->
+    </gazebo>
+    <gazebo reference="FL_Wheel">
+        <material>
+            <color rgba="0.792156862745098 0.819607843137255 0.933333333333333 1" />
+        </material>
+        <!-- Arbitrary friction values -->
+        <mu1 value="0.001"/>
+        <mu2 value="0.001"/>
+    </gazebo>
+    <gazebo reference="ML_Wheel">
+        <material>
+            <color rgba="0.792156862745098 0.819607843137255 0.933333333333333 1" />
+        </material>
+        <!-- Arbitrary friction values -->
+        <mu1 value="0.001"/>
+        <mu2 value="0.001"/>
+    </gazebo>
+    <gazebo reference="BL_Wheel">
+        <material>
+            <color rgba="0.792156862745098 0.819607843137255 0.933333333333333 1" />
+        </material>
+        <!-- Arbitrary friction values -->
+        <mu1 value="0.001"/>
+        <mu2 value="0.001"/>
+    </gazebo>
+    <gazebo reference="TL_Wheel">
+        <material>
+            <color rgba="0.792156862745098 0.819607843137255 0.933333333333333 1" />
+        </material>
+        <!-- Arbitrary friction values -->
+        <mu1 value="0.001"/>
+        <mu2 value="0.001"/>
+    </gazebo>
+    <gazebo reference="FR_Wheel">
+        <material>
+            <color rgba="0.792156862745098 0.819607843137255 0.933333333333333 1" />
+        </material>
+        <!-- Arbitrary friction values -->
+        <mu1 value="0.001"/>
+        <mu2 value="0.001"/>
+    </gazebo>
+    <gazebo reference="MR_Wheel">
+        <material>
+            <color rgba="0.792156862745098 0.819607843137255 0.933333333333333 1" />
+        </material>
+        <!-- Arbitrary friction values -->
+        <mu1 value="0.001"/>
+        <mu2 value="0.001"/>
+    </gazebo>
+    <gazebo reference="BR_Wheel">
+        <material>
+            <color rgba="0.792156862745098 0.819607843137255 0.933333333333333 1" />
+        </material>
+        <!-- Arbitrary friction values -->
+        <mu1 value="0.001"/>
+        <mu2 value="0.001"/>
+    </gazebo>
+    <gazebo reference="TR_Wheel">
+        <material>
+            <color rgba="0.792156862745098 0.819607843137255 0.933333333333333 1" />
+        </material>
+        <!-- Arbitrary friction values -->
+        <mu1 value="0.001"/>
+        <mu2 value="0.001"/>
     </gazebo>
     <!-- Define Gazebo info for any sensors -->

Commit message: Updated the gazebo components of the URDF to (hopefully) be more up to date with new Gazebo standards

File: ros2/description/urdf/gazebo.xacro (robot description, xacro)
@@ -11,127 +11,171 @@
     </gazebo>
     <gazebo reference="DL_Wheel">
-        <material>
-            <color rgba="0.79216 0.81961 0.93333 1" />
-        </material>
-        <!-- Arbitrary friction values -->
-        <mu1 value="0.001"/>
-        <mu2 value="0.001"/>
+        <material>Gazebo/SkyBlue</material>
+        <collision>
+            <surface>
+                <friction>
+                    <ode>
+                        <mu>0.001</mu>
+                        <mu2>0.001</mu2>
+                    </ode>
+                </friction>
+            </surface>
+        </collision>
     </gazebo>
     <gazebo reference="DR_Wheel">
-        <material>
-            <color rgba="0.792156862745098 0.819607843137255 0.933333333333333 1" />
-        </material>
-        <!-- Arbitrary friction values -->
-        <mu1 value="0.001"/>
-        <mu2 value="0.001"/>
+        <material>Gazebo/SkyBlue</material>
+        <collision>
+            <surface>
+                <friction>
+                    <ode>
+                        <mu>0.001</mu>
+                        <mu2>0.001</mu2>
+                    </ode>
+                </friction>
+            </surface>
+        </collision>
     </gazebo>
     <gazebo reference="BLA">
-        <material>
-            <color rgba="0.792156862745098 0.819607843137255 0.933333333333333 1" />
-        </material>
+        <material>Gazebo/SkyBlue</material>
         <!-- TODO: Any other configurations for Linear Actuators -->
     </gazebo>
     <gazebo reference="LA">
-        <material>
-            <color rgba="0.792156862745098 0.819607843137255 0.933333333333333 1" />
-        </material>
+        <material>Gazebo/SkyBlue</material>
         <!-- TODO: Any other configurations for Linear Actuators -->
     </gazebo>
     <!-- Not sure if this is a wheel or a linear actuator -->
     <gazebo reference="TLA">
-        <material>
-            <color rgba="0.792156862745098 0.819607843137255 0.933333333333333 1" />
-        </material>
+        <material>Gazebo/SkyBlue</material>
         <!-- Included in case its a wheel -->
-        <mu1 value="0.001"/>
-        <mu2 value="0.001"/>
+        <collision>
+            <surface>
+                <friction>
+                    <ode>
+                        <mu>0.001</mu>
+                        <mu2>0.001</mu2>
+                    </ode>
+                </friction>
+            </surface>
+        </collision>
     </gazebo>
     <gazebo reference="Hopper">
-        <material>
-            <color rgba="0.866666666666667 0.909803921568627 1 1" />
-        </material>
+        <material>Gazebo/White</material>
         <!-- TODO: Any other configurations for the Hopper -->
     </gazebo>
     <gazebo reference="Hopper_Door">
-        <material>
-            <color rgba="0.866666666666667 0.909803921568627 1 1" />
-        </material>
+        <material>Gazebo/White</material>
         <!-- TODO: Any other configurations for the Hopper Door -->
     </gazebo>
     <gazebo reference="Hopper_Latch">
-        <material>
-            <color rgba="1 0 1 1" />
-        </material>
+        <material>Gazebo/Purple</material>
         <!-- TODO: Any other configurations for the Hopper Latch -->
     </gazebo>
     <gazebo reference="Excavation">
-        <material>
-            <color rgba="0.792156862745098 0.819607843137255 0.933333333333333 1" />
-        </material>
+        <material>Gazebo/SkyBlue</material>
         <!-- TODO: Any other configurations for Excavation -->
     </gazebo>
     <gazebo reference="FL_Wheel">
-        <material>
-            <color rgba="0.792156862745098 0.819607843137255 0.933333333333333 1" />
-        </material>
-        <!-- Arbitrary friction values -->
-        <mu1 value="0.001"/>
-        <mu2 value="0.001"/>
+        <material>Gazebo/SkyBlue</material>
+        <collision>
+            <surface>
+                <friction>
+                    <ode>
+                        <mu>0.001</mu>
+                        <mu2>0.001</mu2>
+                    </ode>
+                </friction>
+            </surface>
+        </collision>
     </gazebo>
     <gazebo reference="ML_Wheel">
-        <material>
-            <color rgba="0.792156862745098 0.819607843137255 0.933333333333333 1" />
-        </material>
-        <!-- Arbitrary friction values -->
-        <mu1 value="0.001"/>
-        <mu2 value="0.001"/>
+        <material>Gazebo/SkyBlue</material>
+        <collision>
+            <surface>
+                <friction>
+                    <ode>
+                        <mu>0.001</mu>
+                        <mu2>0.001</mu2>
+                    </ode>
+                </friction>
+            </surface>
+        </collision>
     </gazebo>
     <gazebo reference="BL_Wheel">
-        <material>
-            <color rgba="0.792156862745098 0.819607843137255 0.933333333333333 1" />
-        </material>
-        <!-- Arbitrary friction values -->
-        <mu1 value="0.001"/>
-        <mu2 value="0.001"/>
+        <material>Gazebo/SkyBlue</material>
+        <collision>
+            <surface>
+                <friction>
+                    <ode>
+                        <mu>0.001</mu>
+                        <mu2>0.001</mu2>
+                    </ode>
+                </friction>
+            </surface>
+        </collision>
     </gazebo>
     <gazebo reference="TL_Wheel">
-        <material>
-            <color rgba="0.792156862745098 0.819607843137255 0.933333333333333 1" />
-        </material>
-        <!-- Arbitrary friction values -->
-        <mu1 value="0.001"/>
-        <mu2 value="0.001"/>
+        <material>Gazebo/SkyBlue</material>
+        <collision>
+            <surface>
+                <friction>
+                    <ode>
+                        <mu>0.001</mu>
+                        <mu2>0.001</mu2>
+                    </ode>
+                </friction>
+            </surface>
+        </collision>
     </gazebo>
     <gazebo reference="FR_Wheel">
-        <material>
-            <color rgba="0.792156862745098 0.819607843137255 0.933333333333333 1" />
-        </material>
-        <!-- Arbitrary friction values -->
-        <mu1 value="0.001"/>
-        <mu2 value="0.001"/>
+        <material>Gazebo/SkyBlue</material>
+        <collision>
+            <surface>
+                <friction>
+                    <ode>
+                        <mu>0.001</mu>
+                        <mu2>0.001</mu2>
+                    </ode>
+                </friction>
+            </surface>
+        </collision>
     </gazebo>
     <gazebo reference="MR_Wheel">
-        <material>
-            <color rgba="0.792156862745098 0.819607843137255 0.933333333333333 1" />
-        </material>
-        <!-- Arbitrary friction values -->
-        <mu1 value="0.001"/>
-        <mu2 value="0.001"/>
+        <material>Gazebo/SkyBlue</material>
+        <collision>
+            <surface>
+                <friction>
+                    <ode>
+                        <mu>0.001</mu>
+                        <mu2>0.001</mu2>
+                    </ode>
+                </friction>
+            </surface>
+        </collision>
     </gazebo>
     <gazebo reference="BR_Wheel">
-        <material>
-            <color rgba="0.792156862745098 0.819607843137255 0.933333333333333 1" />
-        </material>
-        <!-- Arbitrary friction values -->
-        <mu1 value="0.001"/>
-        <mu2 value="0.001"/>
+        <material>Gazebo/SkyBlue</material>
+        <collision>
+            <surface>
+                <friction>
+                    <ode>
+                        <mu>0.001</mu>
+                        <mu2>0.001</mu2>
+                    </ode>
+                </friction>
+            </surface>
+        </collision>
     </gazebo>
     <gazebo reference="TR_Wheel">
-        <material>
-            <color rgba="0.792156862745098 0.819607843137255 0.933333333333333 1" />
-        </material>
-        <!-- Arbitrary friction values -->
-        <mu1 value="0.001"/>
-        <mu2 value="0.001"/>
+        <material>Gazebo/SkyBlue</material>
+        <collision>
+            <surface>
+                <friction>
+                    <ode>
+                        <mu>0.001</mu>
+                        <mu2>0.001</mu2>
+                    </ode>
+                </friction>
+            </surface>
+        </collision>
     </gazebo>
     <!-- Define Gazebo info for any sensors -->

Commit message: every part of the URDF now has a distinct color, colors are now (numerically) consistent between gazebo and RVIZ. They dont appear very consistent though because gazebo is dumb and doesnt render colors the same way

File: ros2/description/urdf/gazebo.xacro (robot description, xacro)
@@ -3,13 +3,19 @@
     <!-- Add any Gazebo references to links/joints including color and friction values -->
     <gazebo reference="chassis_link">
-        <material>Gazebo/White</material>
+        <material>
+            <ambient>0.35 0.35 0.38 1</ambient>
+        </material>
     </gazebo>
     <gazebo reference="Castor">
-        <material>Gazebo/Blue</material>
+        <material>
+            <ambient>1 1 1 1</ambient>
+        </material>
         <mu1 value="0.0"/>  <!-- This is friction -->
         <mu2 value="0.0"/>
     </gazebo>
     <gazebo reference="DL_Wheel">
-        <material>Gazebo/SkyBlue</material>
+        <material>
+            <ambient>0.00 0.60 1.00 1</ambient>
+        </material>
         <collision>
             <surface>
@@ -24,5 +30,7 @@
     </gazebo>
     <gazebo reference="DR_Wheel">
-        <material>Gazebo/SkyBlue</material>
+        <material>
+            <ambient>0.00 0.85 0.40 1</ambient>
+        </material>
         <collision>
             <surface>
@@ -37,14 +45,20 @@
     </gazebo>
     <gazebo reference="BLA">
-        <material>Gazebo/SkyBlue</material>
+        <material>
+            <ambient>0.65 0.45 0.20 1</ambient>
+        </material>
         <!-- TODO: Any other configurations for Linear Actuators -->
     </gazebo>
     <gazebo reference="LA">
-        <material>Gazebo/SkyBlue</material>
+        <material>
+            <ambient>1.00 0.08 0.58 1</ambient>
+        </material>
         <!-- TODO: Any other configurations for Linear Actuators -->
     </gazebo>
     <!-- Not sure if this is a wheel or a linear actuator -->
     <gazebo reference="TLA">
-        <material>Gazebo/SkyBlue</material>
+        <material>
+            <ambient>1.00 0.85 0.00 1</ambient>
+        </material>
         <!-- Included in case its a wheel -->
         <collision>
@@ -60,21 +74,31 @@
     </gazebo>
     <gazebo reference="Hopper">
-        <material>Gazebo/White</material>
+        <material>
+            <ambient>0.55 0.62 0.68 1</ambient>
+        </material>
         <!-- TODO: Any other configurations for the Hopper -->
     </gazebo>
     <gazebo reference="Hopper_Door">
-        <material>Gazebo/White</material>
+        <material>
+            <ambient>0.60 0.40 0.65 1</ambient>
+        </material>
         <!-- TODO: Any other configurations for the Hopper Door -->
     </gazebo>
     <gazebo reference="Hopper_Latch">
-        <material>Gazebo/Purple</material>
+        <material>
+            <ambient>1.00 0.27 0.00 1</ambient>
+        </material>
         <!-- TODO: Any other configurations for the Hopper Latch -->
     </gazebo>
     <gazebo reference="Excavation">
-        <material>Gazebo/SkyBlue</material>
+        <material>
+            <ambient>0.00 1.00 0.80 1</ambient>
+        </material>
         <!-- TODO: Any other configurations for Excavation -->
     </gazebo>
     <gazebo reference="FL_Wheel">
-        <material>Gazebo/SkyBlue</material>
+        <material>
+            <ambient>0.95 0.20 0.20 1</ambient>
+        </material>
         <collision>
             <surface>
@@ -89,5 +113,7 @@
     </gazebo>
     <gazebo reference="ML_Wheel">
-        <material>Gazebo/SkyBlue</material>
+        <material>
+            <ambient>0.10 0.70 0.90 1</ambient>
+        </material>
         <collision>
             <surface>
@@ -102,5 +128,7 @@
     </gazebo>
     <gazebo reference="BL_Wheel">
-        <material>Gazebo/SkyBlue</material>
+        <material>
+            <ambient>0.80 0.00 0.80 1</ambient>
+        </material>
         <collision>
             <surface>
@@ -115,5 +143,7 @@
     </gazebo>
     <gazebo reference="TL_Wheel">
-        <material>Gazebo/SkyBlue</material>
+        <material>
+            <ambient>0.10 0.45 1.00 1</ambient>
+        </material>
         <collision>
             <surface>
@@ -128,5 +158,7 @@
     </gazebo>
     <gazebo reference="FR_Wheel">
-        <material>Gazebo/SkyBlue</material>
+        <material>
+            <ambient>1.00 0.55 0.00 1</ambient>
+        </material>
         <collision>
             <surface>
@@ -141,5 +173,7 @@
     </gazebo>
     <gazebo reference="MR_Wheel">
-        <material>Gazebo/SkyBlue</material>
+        <material>
+            <ambient>0.20 0.90 0.50 1</ambient>
+        </material>
         <collision>
             <surface>
@@ -154,5 +188,7 @@
     </gazebo>
     <gazebo reference="BR_Wheel">
-        <material>Gazebo/SkyBlue</material>
+        <material>
+            <ambient>0.70 0.20 1.00 1</ambient>
+        </material>
         <collision>
             <surface>
@@ -167,5 +203,7 @@
     </gazebo>
     <gazebo reference="TR_Wheel">
-        <material>Gazebo/SkyBlue</material>
+        <material>
+            <ambient>0.00 0.90 0.70 1</ambient>
+        </material>
         <collision>
             <surface>

File: ros2/description/urdf/tibble_core.xacro (robot description, xacro)
@@ -31,5 +31,5 @@
         name="">
         <color
-          rgba="0.25098 0.25098 0.25098 1" />
+          rgba="0.35 0.35 0.38 1" />
       </material>
     </visual>
@@ -82,5 +82,5 @@
         name="">
         <color
-          rgba="0.79216 0.81961 0.93333 1" />
+          rgba="0.00 0.60 1.00 1" />
       </material>
     </visual>
@@ -135,5 +135,5 @@
         name="">
         <color
-          rgba="0.792156862745098 0.819607843137255 0.933333333333333 1" />
+          rgba="0.00 0.85 0.40 1" />
       </material>
     </visual>
@@ -188,5 +188,5 @@
         name="">
         <color
-          rgba="0.792156862745098 0.819607843137255 0.933333333333333 1" />
+          rgba="0.65 0.45 0.20 1" />
       </material>
     </visual>
@@ -246,5 +246,5 @@
         name="">
         <color
-          rgba="0.792156862745098 0.819607843137255 0.933333333333333 1" />
+          rgba="1.00 0.08 0.58 1" />
       </material>
     </visual>
@@ -304,5 +304,5 @@
         name="">
         <color
-          rgba="0.792156862745098 0.819607843137255 0.933333333333333 1" />
+          rgba="1.00 0.85 0.00 1" />
       </material>
     </visual>
@@ -362,5 +362,5 @@
         name="">
         <color
-          rgba="0.866666666666667 0.909803921568627 1 1" />
+          rgba="0.55 0.62 0.68 1" />
       </material>
     </visual>
@@ -420,5 +420,5 @@
         name="">
         <color
-          rgba="0.866666666666667 0.909803921568627 1 1" />
+          rgba="0.60 0.40 0.65 1" />
       </material>
     </visual>
@@ -478,5 +478,5 @@
         name="">
         <color
-          rgba="1 0 1 1" />
+          rgba="1.00 0.27 0.00 1" />
       </material>
     </visual>
@@ -536,5 +536,5 @@
         name="">
         <color
-          rgba="0.792156862745098 0.819607843137255 0.933333333333333 1" />
+          rgba="0.00 1.00 0.80 1" />
       </material>
     </visual>
@@ -589,5 +589,5 @@
         name="">
         <color
-          rgba="0.792156862745098 0.819607843137255 0.933333333333333 1" />
+          rgba="0.95 0.20 0.20 1" />
       </material>
     </visual>
@@ -642,5 +642,5 @@
         name="">
         <color
-          rgba="0.792156862745098 0.819607843137255 0.933333333333333 1" />
+          rgba="0.10 0.70 0.90 1" />
       </material>
     </visual>
@@ -695,5 +695,5 @@
         name="">
         <color
-          rgba="0.792156862745098 0.819607843137255 0.933333333333333 1" />
+          rgba="0.80 0.00 0.80 1" />
       </material>
     </visual>
@@ -748,5 +748,5 @@
         name="">
         <color
-          rgba="0.792156862745098 0.819607843137255 0.933333333333333 1" />
+          rgba="0.10 0.45 1.00 1" />
       </material>
     </visual>
@@ -801,5 +801,5 @@
         name="">
         <color
-          rgba="0.792156862745098 0.819607843137255 0.933333333333333 1" />
+          rgba="1.00 0.55 0.00 1" />
       </material>
     </visual>
@@ -854,5 +854,5 @@
         name="">
         <color
-          rgba="0.792156862745098 0.819607843137255 0.933333333333333 1" />
+          rgba="0.20 0.90 0.50 1" />
       </material>
     </visual>
@@ -907,5 +907,5 @@
         name="">
         <color
-          rgba="0.792156862745098 0.819607843137255 0.933333333333333 1" />
+          rgba="0.70 0.20 1.00 1" />
       </material>
     </visual>
@@ -960,5 +960,5 @@
         name="">
         <color
-          rgba="1 1 1 1" />
+          rgba="0.00 0.90 0.70 1" />
       </material>
     </visual>
