Commit message: Added teleop to simulation. Removed collison from everything but the wheels to keep the sim bot from getting stuck. Very dirty implementation but it almost works.
Currently the robot teleop breaks after about 1 minute and 10 seconds every time  the simulation runs. Possibly a timeout issue.

File: ros2/description/urdf/gazebo.xacro (robot description, xacro)
@@ -11,6 +11,14 @@
             <ambient>1 1 1 1</ambient>
         </material>
-        <mu1 value="0.0"/>  <!-- This is friction -->
-        <mu2 value="0.0"/>
+        <collision>
+            <surface>
+                <friction>
+                    <ode>
+                        <mu>0.0001</mu> <!-- This is friction -->
+                        <mu2>0.0001</mu2>
+                    </ode>
+                </friction>
+            </surface>
+        </collision>
     </gazebo>
     <gazebo reference="DL_Wheel">
@@ -22,6 +30,6 @@
                 <friction>
                     <ode>
-                        <mu>0.001</mu>
-                        <mu2>0.001</mu2>
+                        <mu>0.0001</mu>
+                        <mu2>0.0001</mu2>
                     </ode>
                 </friction>
@@ -37,6 +45,6 @@
                 <friction>
                     <ode>
-                        <mu>0.001</mu>
-                        <mu2>0.001</mu2>
+                        <mu>0.0001</mu>
+                        <mu2>0.0001</mu2>
                     </ode>
                 </friction>
@@ -66,6 +74,6 @@
                 <friction>
                     <ode>
-                        <mu>0.001</mu>
-                        <mu2>0.001</mu2>
+                        <mu>1.0</mu>
+                        <mu2>0.1</mu2>
                     </ode>
                 </friction>
@@ -105,21 +113,25 @@
                 <friction>
                     <ode>
-                        <mu>0.001</mu>
-                        <mu2>0.001</mu2>
-                    </ode>
-                </friction>
-            </surface>
-        </collision>
+                        <mu>0.0001</mu>
+                        <mu2>0.0001</mu2>
+                    </ode>
+                </friction>
+            </surface>
+        </collision>
+    </gazebo>
+    <gazebo reference="FL_Wheel_Rotate">
+        <implicitSpringDamper>true</implicitSpringDamper>
+        <dynamics damping="0.01" friction="0.0"/>
     </gazebo>
     <gazebo reference="ML_Wheel">
         <material>
-            <ambient>0.10 0.70 0.90 1</ambient>
-        </material>
-        <collision>
-            <surface>
-                <friction>
-                    <ode>
-                        <mu>0.001</mu>
-                        <mu2>0.001</mu2>
+            <ambient>0.50 0.70 0.90 1</ambient>
+        </material>
+        <collision>
+            <surface>
+                <friction>
+                    <ode>
+                        <mu>1.0</mu>
+                        <mu2>0.5</mu2>
                     </ode>
                 </friction>
@@ -135,21 +147,25 @@
                 <friction>
                     <ode>
-                        <mu>0.001</mu>
-                        <mu2>0.001</mu2>
-                    </ode>
-                </friction>
-            </surface>
-        </collision>
+                        <mu>0.0001</mu>
+                        <mu2>0.0001</mu2>
+                    </ode>
+                </friction>
+            </surface>
+        </collision>
+    </gazebo>
+    <gazebo reference="BL_Wheel_Rotate">
+        <implicitSpringDamper>true</implicitSpringDamper>
+        <dynamics damping="0.01" friction="0.0"/>
     </gazebo>
     <gazebo reference="TL_Wheel">
         <material>
-            <ambient>0.10 0.45 1.00 1</ambient>
-        </material>
-        <collision>
-            <surface>
-                <friction>
-                    <ode>
-                        <mu>0.001</mu>
-                        <mu2>0.001</mu2>
+            <ambient>0.50 0.45 1.00 1</ambient>
+        </material>
+        <collision>
+            <surface>
+                <friction>
+                    <ode>
+                        <mu>0.0001</mu>
+                        <mu2>0.0001</mu2>
                     </ode>
                 </friction>
@@ -165,10 +181,14 @@
                 <friction>
                     <ode>
-                        <mu>0.001</mu>
-                        <mu2>0.001</mu2>
-                    </ode>
-                </friction>
-            </surface>
-        </collision>
+                        <mu>0.0001</mu>
+                        <mu2>0.0001</mu2>
+                    </ode>
+                </friction>
+            </surface>
+        </collision>
+    </gazebo>
+    <gazebo reference="FR_Wheel_Rotate">
+        <implicitSpringDamper>true</implicitSpringDamper>
+        <dynamics damping="0.01" friction="0.0"/>
     </gazebo>
     <gazebo reference="MR_Wheel">
@@ -180,6 +200,6 @@
                 <friction>
                     <ode>
-                        <mu>0.001</mu>
-                        <mu2>0.001</mu2>
+                        <mu>1.0</mu>
+                        <mu2>0.5</mu2>
                     </ode>
                 </friction>
@@ -195,10 +215,14 @@
                 <friction>
                     <ode>
-                        <mu>0.001</mu>
-                        <mu2>0.001</mu2>
-                    </ode>
-                </friction>
-            </surface>
-        </collision>
+                        <mu>0.0001</mu>
+                        <mu2>0.0001</mu2>
+                    </ode>
+                </friction>
+            </surface>
+        </collision>
+    </gazebo>
+    <gazebo reference="BR_Wheel_Rotate">
+        <implicitSpringDamper>true</implicitSpringDamper>
+        <dynamics damping="0.01" friction="0.0"/>
     </gazebo>
     <gazebo reference="TR_Wheel">
@@ -210,6 +234,6 @@
                 <friction>
                     <ode>
-                        <mu>0.001</mu>
-                        <mu2>0.001</mu2>
+                        <mu>0.0001</mu>
+                        <mu2>0.0001</mu2>
                     </ode>
                 </friction>

File: ros2/description/urdf/tibble_core.xacro (robot description, xacro)
@@ -34,5 +34,5 @@
       </material>
     </visual>
-    <collision>
+    <!-- <collision>
       <origin
         xyz="0 0 0"
@@ -42,5 +42,5 @@
           filename="file://$(find description)/meshes/Chassis.STL" />
       </geometry>
-    </collision>
+    </collision> -->
   </link>
   <joint
@@ -85,5 +85,5 @@
       </material>
     </visual>
-    <collision>
+    <!-- <collision>
       <origin
         xyz="0 0 0"
@@ -93,5 +93,5 @@
           filename="file://$(find description)/meshes/DL_Wheel.STL" />
       </geometry>
-    </collision>
+    </collision> -->
   </link>
   <joint
@@ -138,5 +138,5 @@
       </material>
     </visual>
-    <collision>
+    <!-- <collision>
       <origin
         xyz="0 0 0"
@@ -146,5 +146,5 @@
           filename="file://$(find description)/meshes/DR_Wheel.STL" />
       </geometry>
-    </collision>
+    </collision> -->
   </link>
   <joint
@@ -191,5 +191,5 @@
       </material>
     </visual>
-    <collision>
+    <!-- <collision>
       <origin
         xyz="0 0 0"
@@ -199,5 +199,5 @@
           filename="file://$(find description)/meshes/BLA.STL" />
       </geometry>
-    </collision>
+    </collision> -->
   </link>
   <joint
@@ -249,5 +249,5 @@
       </material>
     </visual>
-    <collision>
+    <!-- <collision>
       <origin
         xyz="0 0 0"
@@ -257,5 +257,5 @@
           filename="file://$(find description)/meshes/LA.STL" />
       </geometry>
-    </collision>
+    </collision> -->
   </link>
   <joint
@@ -307,5 +307,5 @@
       </material>
     </visual>
-    <collision>
+    <!-- <collision>
       <origin
         xyz="0 0 0"
@@ -315,5 +315,5 @@
           filename="file://$(find description)/meshes/TLA.STL" />
       </geometry>
-    </collision>
+    </collision> -->
   </link>
   <joint
@@ -365,5 +365,5 @@
       </material>
     </visual>
-    <collision>
+    <!-- <collision>
       <origin
         xyz="0 0 0"
@@ -373,5 +373,5 @@
           filename="file://$(find description)/meshes/Hopper.STL" />
       </geometry>
-    </collision>
+    </collision> -->
   </link>
   <joint
@@ -423,5 +423,5 @@
       </material>
     </visual>
-    <collision>
+    <!-- <collision>
       <origin
         xyz="0 0 0"
@@ -431,5 +431,5 @@
           filename="file://$(find description)/meshes/Hopper_Door.STL" />
       </geometry>
-    </collision>
+    </collision> -->
   </link>
   <joint
@@ -481,5 +481,5 @@
       </material>
     </visual>
-    <collision>
+    <!-- <collision>
       <origin
         xyz="0 0 0"
@@ -489,5 +489,5 @@
           filename="file://$(find description)/meshes/Hopper_Latch.STL" />
       </geometry>
-    </collision>
+    </collision> -->
   </link>
   <joint
@@ -599,5 +599,5 @@
         <!-- <mesh
           filename="file://$(find description)/meshes/FL_Wheel.STL" /> -->
-          <sphere radius="0.0929"/>
+          <sphere radius="0.076835"/>
       </geometry>
     </collision>
@@ -615,4 +615,5 @@
     <axis
       xyz="0 0 -1" />
+    <dynamics damping="0.001" friction="0.0"/>
   </joint>
   <link
@@ -653,5 +654,5 @@
         <!-- <mesh
           filename="file://$(find description)/meshes/ML_Wheel.STL" /> -->
-          <sphere radius="0.0929"/>
+          <sphere radius="0.076835"/>
       </geometry>
     </collision>
@@ -707,5 +708,5 @@
         <!-- <mesh
           filename="file://$(find description)/meshes/BL_Wheel.STL" /> -->
-          <sphere radius="0.0929"/>
+          <sphere radius="0.076835"/>
       </geometry>
     </collision>
@@ -723,4 +724,5 @@
     <axis
       xyz="0 0 -1" />
+    <dynamics damping="0.001" friction="0.0"/>
   </joint>
   <link
@@ -754,5 +756,5 @@
       </material>
     </visual>
-    <collision>
+    <!-- <collision>
       <origin
         xyz="0 0 0"
@@ -762,5 +764,5 @@
           filename="file://$(find description)/meshes/TL_Wheel.STL" />
       </geometry>
-    </collision>
+    </collision> -->
   </link>
   <joint
@@ -814,5 +816,5 @@
         <!-- <mesh
           filename="file://$(find description)/meshes/FR_Wheel.STL" /> -->
-          <sphere radius="0.0929"/>
+          <sphere radius="0.076835"/>
       </geometry>
     </collision>
@@ -830,4 +832,5 @@
     <axis
       xyz="0 0 -1" />
+    <dynamics damping="0.001" friction="0.0"/>
   </joint>
   <link
@@ -868,5 +871,5 @@
         <!-- <mesh
           filename="file://$(find description)/meshes/MR_Wheel.STL" /> -->
-          <sphere radius="0.0929"/>
+          <sphere radius="0.076835"/>
       </geometry>
     </collision>
@@ -922,5 +925,5 @@
         <!-- <mesh
           filename="file://$(find description)/meshes/BR_Wheel.STL" /> -->
-          <sphere radius="0.0929"/>
+          <sphere radius="0.076835"/>
       </geometry>
     </collision>
@@ -938,4 +941,5 @@
     <axis
       xyz="0 0 -1" />
+    <dynamics damping="0.001" friction="0.0"/>
   </joint>
   <link
@@ -969,5 +973,5 @@
       </material>
     </visual>
-    <collision>
+    <!-- <collision>
       <origin
         xyz="0 0 0"
@@ -977,5 +981,5 @@
           filename="file://$(find description)/meshes/TR_Wheel.STL" />
       </geometry>
-    </collision>
+    </collision> -->
   </link>
   <joint

Commit message: Add LaserScan

File: ros2/description/urdf/gazebo.xacro (robot description, xacro)
@@ -241,27 +241,3 @@
         </collision>
     </gazebo>
-    <!-- Define Gazebo info for any sensors -->
-    <gazebo reference="laser_frame">
-        <material>Gazebo/Red</material>
-        <sensor name="laser" type="gpu_lidar">
-            <pose> 0 0 0 0 0 0 </pose>
-            <visualize>true</visualize>
-            <update_rate>10</update_rate>
-            <lidar>
-                <scan>
-                    <horizontal>
-                        <samples>360</samples>
-                        <min_angle>-3.14</min_angle>
-                        <max_angle>3.14</max_angle>
-                    </horizontal>
-                </scan>
-                <range>
-                    <min>0.3</min>
-                    <max>12</max>
-                </range>
-            </lidar>
-            <topic>scan</topic>
-            <gz_frame_id>laser_frame</gz_frame_id>
-        </sensor>
-    </gazebo>
 </robot>

File: ros2/description/urdf/sensors.xacro (robot description, xacro)
@@ -2,3 +2,51 @@
 <robot xmlns:xacro="http://www.ros.org/wiki/xacro">
     <!-- Define the joint/link for the sensors -->
+    <joint name="lidar_joint" type="fixed">
+        <parent link="base_link"/>
+        <child link="laser_frame"/>
+        <origin xyz="0 0.3 0" rpy="${pi/2} 0 0"/>
+    </joint>
+    <link name="laser_frame">
+        <visual>
+            <geometry>
+                <cylinder radius="0.05" length="0.04"/>
+            </geometry>
+            <material name="red"/>
+        </visual>
+        <collision>
+            <geometry>
+                <cylinder radius="0.05" length="0.04"/>
+            </geometry>
+        </collision>
+        <inertial>
+            <origin xyz="0 0 0" rpy="0 0 0"/>
+            <mass value="0.1" />
+            <inertia ixx="${(1/12) * 0.1 * (3*0.05*0.05 + 0.04*0.04)}" ixy="0.0" ixz="0.0"
+                    iyy="${(1/12) * 0.1 * (3*0.05*0.05 + 0.04*0.04)}" iyz="0.0"
+                    izz="${(1/2) * 0.1 * (0.05*0.05)}" />
+        </inertial>
+    </link>
+    <gazebo reference="laser_frame">
+        <material>Gazebo/Red</material>
+        <sensor name="laser" type="gpu_lidar">
+            <pose> 0 0 0 0 0 0 </pose>
+            <visualize>true</visualize>
+            <update_rate>10</update_rate>
+            <lidar>
+                <scan>
+                    <horizontal>
+                        <samples>360</samples>
+                        <min_angle>-3.14</min_angle>
+                        <max_angle>3.14</max_angle>
+                    </horizontal>
+                </scan>
+                <range>
+                    <min>0.3</min>
+                    <max>12</max>
+                </range>
+            </lidar>
+            <topic>scan</topic>
+            <gz_frame_id>laser_frame</gz_frame_id>
+        </sensor>
+    </gazebo>
 </robot>
