Commit message: Added camera (not in correct spot)

File: ros2/description/urdf/sensors.xacro (robot description, xacro)
@@ -2,4 +2,56 @@
 <robot xmlns:xacro="http://www.ros.org/wiki/xacro">
     <!-- Define the joint/link for the sensors -->
+    <!-- CAMERA -->
+    <joint name="camera_joint" type="fixed">
+        <parent link="base_link"/>
+        <child link="camera_link"/>
+        <origin xyz="0 0.27 0" rpy="-${pi/2} -${pi/2} 0"/>
+    </joint>
+    <!-- The camera is represented by a simple box and cylinder floating above the bot-->
+    <link name="camera_link">
+        <visual>
+            <geometry>
+                <box size="0.010 0.03 0.03"/>
+            </geometry>
+            <material name="red"/>
+        </visual>
+        <visual>
+            <origin xyz="0 0 -0.05"/>
+            <geometry>
+                <cylinder radius="0.002" length="0.1"/>
+            </geometry>
+            <material name="red"/>
+        </visual>
+    </link>
+    <joint name="camera_optical_joint" type="fixed">
+        <parent link="camera_link"/>
+        <child link="camera_link_optical"/>
+        <origin xyz="0.1 0 0" rpy="0 0 0"/>
+    </joint>
+    <link name="camera_link_optical"></link>
+    <gazebo reference="camera_link">
+        <material>Gazebo/Red</material>
+        <sensor name="rgbd_camera" type="rgbd_camera">
+            <pose> 0 0 0 0 0 0 </pose>
+            <visualize>true</visualize>
+            <update_rate>10</update_rate>
+            <camera>
+                <camera_info_topic>camera/camera_info</camera_info_topic>
+                <horizontal_fov>1.089</horizontal_fov>
+                <image>
+                    <format>R8G8B8</format>
+                    <width>640</width>
+                    <height>480</height>
+                </image>
+                <clip>
+                    <near>0.05</near>
+                    <far>8.0</far>
+                </clip>
+            </camera>
+            <topic>camera</topic>
+            <gz_frame_id>camera_link_optical</gz_frame_id>
+        </sensor>
+    </gazebo>
+    <!-- LIDAR -->
     <joint name="lidar_joint" type="fixed">
         <parent link="base_link"/>

Commit message: Add sensors

File: ros2/description/urdf/sensors.xacro (robot description, xacro)
@@ -2,3 +2,103 @@
 <robot xmlns:xacro="http://www.ros.org/wiki/xacro">
     <!-- Define the joint/link for the sensors -->
+    <!-- Camera -->
+    <joint name="camera_joint" type="fixed">
+        <parent link="base_link"/>
+        <child link="camera_link"/>
+        <origin xyz="0 0.27 0" rpy="-${pi/2} -${pi/2} 0"/>
+    </joint>
+    <!-- The camera is represented by a simple box and cylinder floating above the bot-->
+    <link name="camera_link">
+        <visual>
+            <geometry>
+                <box size="0.010 0.03 0.03"/>
+            </geometry>
+            <material name="red"/>
+        </visual>
+        <visual>
+            <origin xyz="0 0 -0.05"/>
+            <geometry>
+                <cylinder radius="0.002" length="0.1"/>
+            </geometry>
+            <material name="red"/>
+        </visual>
+    </link>
+    <joint name="camera_optical_joint" type="fixed">
+        <parent link="camera_link"/>
+        <child link="camera_link_optical"/>
+        <origin xyz="0.1 0 0" rpy="0 0 0"/>
+    </joint>
+    <link name="camera_link_optical"></link>
+    <gazebo reference="camera_link">
+        <material>Gazebo/Red</material>
+        <sensor name="rgbd_camera" type="rgbd_camera">
+            <pose> 0 0 0 0 0 0 </pose>
+            <visualize>true</visualize>
+            <update_rate>10</update_rate>
+            <camera>
+                <camera_info_topic>camera/camera_info</camera_info_topic>
+                <horizontal_fov>1.089</horizontal_fov>
+                <image>
+                    <format>R8G8B8</format>
+                    <width>640</width>
+                    <height>480</height>
+                </image>
+                <clip>
+                    <near>0.05</near>
+                    <far>8.0</far>
+                </clip>
+            </camera>
+            <topic>camera</topic>
+            <gz_frame_id>camera_link_optical</gz_frame_id>
+        </sensor>
+    </gazebo>
+    <!-- LiDAR -->
+    <joint name="lidar_joint" type="fixed">
+        <parent link="base_link"/>
+        <child link="laser_frame"/>
+        <origin xyz="0 0.3 0" rpy="${pi/2} 0 0"/>
+    </joint>
+    <link name="laser_frame">
+        <visual>
+            <geometry>
+                <cylinder radius="0.05" length="0.04"/>
+            </geometry>
+            <material name="red"/>
+        </visual>
+        <collision>
+            <geometry>
+                <cylinder radius="0.05" length="0.04"/>
+            </geometry>
+        </collision>
+        <inertial>
+            <origin xyz="0 0 0" rpy="0 0 0"/>
+            <mass value="0.1" />
+            <inertia ixx="${(1/12) * 0.1 * (3*0.05*0.05 + 0.04*0.04)}" ixy="0.0" ixz="0.0"
+                    iyy="${(1/12) * 0.1 * (3*0.05*0.05 + 0.04*0.04)}" iyz="0.0"
+                    izz="${(1/2) * 0.1 * (0.05*0.05)}" />
+        </inertial>
+    </link>
+    <gazebo reference="laser_frame">
+        <material>Gazebo/Red</material>
+        <sensor name="laser" type="gpu_lidar">
+            <pose> 0 0 0 0 0 0 </pose>
+            <visualize>true</visualize>
+            <update_rate>10</update_rate>
+            <lidar>
+                <scan>
+                    <horizontal>
+                        <samples>360</samples>
+                        <min_angle>-3.14</min_angle>
+                        <max_angle>3.14</max_angle>
+                    </horizontal>
+                </scan>
+                <range>
+                    <min>0.3</min>
+                    <max>12</max>
+                </range>
+            </lidar>
+            <topic>scan</topic>
+            <gz_frame_id>laser_frame</gz_frame_id>
+        </sensor>
+    </gazebo>
 </robot>

Commit message: Test realsense2 camera

File: ros2/description/urdf/sensors.xacro (robot description, xacro)
@@ -9,48 +9,5 @@
     </joint>
     <!-- The camera is represented by a simple box and cylinder floating above the bot-->
-    <link name="camera_link">
-        <visual>
-            <geometry>
-                <box size="0.010 0.03 0.03"/>
-            </geometry>
-            <material name="red"/>
-        </visual>
-        <visual>
-            <origin xyz="0 0 -0.05"/>
-            <geometry>
-                <cylinder radius="0.002" length="0.1"/>
-            </geometry>
-            <material name="red"/>
-        </visual>
-    </link>
-    <joint name="camera_optical_joint" type="fixed">
-        <parent link="camera_link"/>
-        <child link="camera_link_optical"/>
-        <origin xyz="0.1 0 0" rpy="0 0 0"/>
-    </joint>
-    <link name="camera_link_optical"></link>
-    <gazebo reference="camera_link">
-        <material>Gazebo/Red</material>
-        <sensor name="rgbd_camera" type="rgbd_camera">
-            <pose> 0 0 0 0 0 0 </pose>
-            <visualize>true</visualize>
-            <update_rate>10</update_rate>
-            <camera>
-                <camera_info_topic>camera/camera_info</camera_info_topic>
-                <horizontal_fov>1.089</horizontal_fov>
-                <image>
-                    <format>R8G8B8</format>
-                    <width>640</width>
-                    <height>480</height>
-                </image>
-                <clip>
-                    <near>0.05</near>
-                    <far>8.0</far>
-                </clip>
-            </camera>
-            <topic>camera</topic>
-            <gz_frame_id>camera_link_optical</gz_frame_id>
-        </sensor>
-    </gazebo>
+    <xacro:include filename="$(find realsense2_description)/urdf/_d435.urdf.xacro" />
     <!-- LiDAR -->
     <joint name="lidar_joint" type="fixed">

Commit message: Try #2

File: ros2/description/urdf/sensors.xacro (robot description, xacro)
@@ -9,5 +9,10 @@
     </joint>
     <!-- The camera is represented by a simple box and cylinder floating above the bot-->
-    <xacro:include filename="$(find realsense2_description)/urdf/_d435.urdf.xacro" />
+    <xacro:sensor_d435 name="camera_front" parent="base_link" use_nominal_extrinsics="true">
+        <origin xyz="0.3 0.0 0.15" rpy="0 0 0"/>
+    </xacro:sensor_d435>
+    <xacro:sensor_d435 name="camera_rear" parent="base_link" use_nominal_extrinsics="true">
+        <origin xyz="-0.3 0.0 0.15" rpy="0 0 3.14159"/>
+    </xacro:sensor_d435>
     <!-- LiDAR -->
     <joint name="lidar_joint" type="fixed">

Commit message: Add realsense camera model in URDF sensors

File: ros2/description/urdf/sensors.xacro (robot description, xacro)
@@ -3,10 +3,4 @@
     <!-- Define the joint/link for the sensors -->
     <!-- Camera -->
-    <joint name="camera_joint" type="fixed">
-        <parent link="base_link"/>
-        <child link="camera_link"/>
-        <origin xyz="0 0.27 0" rpy="-${pi/2} -${pi/2} 0"/>
-    </joint>
-    <!-- The camera is represented by a simple box and cylinder floating above the bot-->
     <xacro:include filename="$(find realsense2_description)/urdf/_d435.urdf.xacro" />
     <xacro:sensor_d435 name="camera_front" parent="base_link" use_nominal_extrinsics="true">

Commit message: Sensors are in the right spot

File: ros2/description/urdf/sensors.xacro (robot description, xacro)
@@ -4,20 +4,20 @@
     <!-- Camera -->
     <xacro:include filename="$(find realsense2_description)/urdf/_d435.urdf.xacro" />
-    <xacro:sensor_d435 name="camera_front" parent="base_link" use_nominal_extrinsics="true">
-        <origin xyz="0.3 0.0 0.15" rpy="0 0 0"/>
+    <xacro:sensor_d435 name="camera_front" parent="Front Camera Fixed" use_nominal_extrinsics="true">
+        <origin xyz="0.02 -0.05 0.03" rpy="0 ${pi} 0"/>
     </xacro:sensor_d435>
-    <xacro:sensor_d435 name="camera_rear" parent="base_link" use_nominal_extrinsics="true">
-        <origin xyz="-0.3 0.0 0.15" rpy="0 0 3.14159"/>
+    <xacro:sensor_d435 name="camera_rear" parent="Back Camera Fixed" use_nominal_extrinsics="true">
+        <origin xyz="0.02 -0.05 0.028" rpy="0 ${pi} 0"/>
     </xacro:sensor_d435>
     <!-- LiDAR -->
     <joint name="lidar_joint" type="fixed">
-        <parent link="base_link"/>
+        <parent link="Lindar Fixed"/>
         <child link="laser_frame"/>
-        <origin xyz="0 0.3 0" rpy="${pi/2} 0 0"/>
+        <origin xyz="0 0.02 0" rpy="${pi/2} 0 0"/>
     </joint>
     <link name="laser_frame">
         <visual>
             <geometry>
-                <cylinder radius="0.05" length="0.04"/>
+                <cylinder radius="0.04" length="0.04"/>
             </geometry>
             <material name="red"/>
@@ -25,5 +25,5 @@
         <collision>
             <geometry>
-                <cylinder radius="0.05" length="0.04"/>
+                <cylinder radius="0.04" length="0.04"/>
             </geometry>
         </collision>
