Commit message: defined joints and interfaces for ros2 control (not sim)

File: ros2/description/urdf/ros2_control.xacro (robot description, xacro)
@@ -3,10 +3,37 @@
     <!-- Load the real robot ROS2 Control information -->
     <xacro:unless value="$(arg sim_mode)">
-        <!-- Almost everything should go in this ros2_control tag -->
-        <ros2_control name="name" type="system">  <!-- This should almost always be system -->
+        <ros2_control name="Tibble" type="system">
             <hardware>  <!-- This defines all the params needed for the hardware component -->
-            <!-- This includes wheel names, which serial device/port to listen to, baud_rate, loop_rate, etc -->
+                <plugin>tibble_hwc/TibbleHWC</plugin>
             </hardware>
             <!-- Define all the joints that will have a command or state interface -->
+            <joint name="DL_Rotate">
+                <command_interface name="velocity">
+                    <param name="min">-10</param>
+                    <param name="max">10</param>
+                </command_interface>
+                <state_interface name="position"/>
+                <state_interface name="velocity"/>
+            </joint>
+            <joint name="DR_Rotate">
+                <command_interface name="velocity">
+                    <param name="min">-10</param>
+                    <param name="max">10</param>
+                </command_interface>
+                <state_interface name="position"/>
+                <state_interface name="velocity"/>
+            </joint>
+            <joint name="LA_Extend">
+                <command_interface name="position"/>
+                <state_interface name="position"/>
+            </joint>
+            <joint name="Excavation_Rotate">
+                <command_interface name="velocity">
+                    <param name="min">-10</param>
+                    <param name="max">10</param>
+                </command_interface>
+                <state_interface name="position"/>
+                <state_interface name="velocity"/>
+            </joint>
         </ros2_control>
     </xacro:unless>
@@ -21,5 +48,5 @@
         <gazebo>
             <plugin name="gz_ros2_control::GazeboSimROS2ControlPlugin" filename="libgz_ros2_control-system.so">
-                <parameters>$(find control)/config/controllersname.yaml</parameters>
+                <parameters>$(find control)/config/tibble_controller.yaml</parameters>
             </plugin>
         </gazebo>

Commit message: Maybe working?

File: ros2/description/urdf/ros2_control.xacro (robot description, xacro)
@@ -53,4 +53,36 @@
             </hardware>
             <!-- Define all joints and their command/state interfaces necessary for sim -->
+            <joint name="FL_Wheel_Rotate">
+                <command_interface name="velocity">
+                    <param name="min">-10</param>
+                    <param name="max">10</param>
+                </command_interface>
+                <state_interface name="velocity"/>
+                <state_interface name="position"/>
+            </joint>
+            <joint name="BL_Wheel_Rotate">
+                <command_interface name="velocity">
+                    <param name="min">-10</param>
+                    <param name="max">10</param>
+                </command_interface>
+                <state_interface name="velocity"/>
+                <state_interface name="position"/>
+            </joint>
+            <joint name="FR_Wheel_Rotate">
+                <command_interface name="velocity">
+                    <param name="min">-10</param>
+                    <param name="max">10</param>
+                </command_interface>
+                <state_interface name="velocity"/>
+                <state_interface name="position"/>
+            </joint>
+            <joint name="BR_Wheel_Rotate">
+                <command_interface name="velocity">
+                    <param name="min">-10</param>
+                    <param name="max">10</param>
+                </command_interface>
+                <state_interface name="velocity"/>
+                <state_interface name="position"/>
+            </joint>
         </ros2_control>
         <gazebo>

Commit message: Add more control joints

File: ros2/description/urdf/ros2_control.xacro (robot description, xacro)
@@ -53,4 +53,108 @@
             </hardware>
             <!-- Define all joints and their command/state interfaces necessary for sim -->
+            <joint name="DL_Rotate">
+                <command_interface name="velocity">
+                    <param name="min">-10</param>
+                    <param name="max">10</param>
+                </command_interface>
+                <state_interface name="velocity"/>
+                <state_interface name="position"/>
+            </joint>
+            <joint name="DR_Rotate">
+                <command_interface name="velocity">
+                    <param name="min">-10</param>
+                    <param name="max">10</param>
+                </command_interface>
+                <state_interface name="velocity"/>
+                <state_interface name="position"/>
+            </joint>
+            <joint name="LLA_Rotate">
+                <command_interface name="velocity">
+                    <param name="min">-10</param>
+                    <param name="max">10</param>
+                </command_interface>
+                <state_interface name="velocity"/>
+                <state_interface name="position"/>
+            </joint>
+            <joint name="LA_Extend">
+                <command_interface name="velocity">
+                    <param name="min">-10</param>
+                    <param name="max">10</param>
+                </command_interface>
+                <state_interface name="velocity"/>
+                <state_interface name="position"/>
+            </joint>
+            <joint name="TLA_Rotate">
+                <command_interface name="velocity">
+                    <param name="min">-10</param>
+                    <param name="max">10</param>
+                </command_interface>
+                <state_interface name="velocity"/>
+                <state_interface name="position"/>
+            </joint>
+            <joint name="Hopper_Rotate">
+                <command_interface name="velocity">
+                    <param name="min">-10</param>
+                    <param name="max">10</param>
+                </command_interface>
+                <state_interface name="velocity"/>
+                <state_interface name="position"/>
+            </joint>
+            <joint name="HopperDoorRotate">
+                <command_interface name="velocity">
+                    <param name="min">-10</param>
+                    <param name="max">10</param>
+                </command_interface>
+                <state_interface name="velocity"/>
+                <state_interface name="position"/>
+            </joint>
+            <joint name="H-Latch_Rotate">
+                <command_interface name="velocity">
+                    <param name="min">-10</param>
+                    <param name="max">10</param>
+                </command_interface>
+                <state_interface name="velocity"/>
+                <state_interface name="position"/>
+            </joint>
+            <joint name="Excavation_Rotate">
+                <command_interface name="velocity">
+                    <param name="min">-10</param>
+                    <param name="max">10</param>
+                </command_interface>
+                <state_interface name="velocity"/>
+                <state_interface name="position"/>
+            </joint>
+            <joint name="ML_Wheel_Rotate">
+                <command_interface name="velocity">
+                    <param name="min">-10</param>
+                    <param name="max">10</param>
+                </command_interface>
+                <state_interface name="velocity"/>
+                <state_interface name="position"/>
+            </joint>
+            <joint name="MR_Wheel_Rotate">
+                <command_interface name="velocity">
+                    <param name="min">-10</param>
+                    <param name="max">10</param>
+                </command_interface>
+                <state_interface name="velocity"/>
+                <state_interface name="position"/>
+            </joint>
+            <joint name="TL_Wheel_Rotate">
+                <command_interface name="velocity">
+                    <param name="min">-10</param>
+                    <param name="max">10</param>
+                </command_interface>
+                <state_interface name="velocity"/>
+                <state_interface name="position"/>
+            </joint>
+            <joint name="TR_Wheel_Rotate">
+                <command_interface name="velocity">
+                    <param name="min">-10</param>
+                    <param name="max">10</param>
+                </command_interface>
+                <state_interface name="velocity"/>
+                <state_interface name="position"/>
+            </joint>
             <joint name="FL_Wheel_Rotate">
                 <command_interface name="velocity">

File: ros2/description/urdf/tibble_core.xacro (robot description, xacro)
@@ -940,5 +940,5 @@
         rpy="0 0 0" />
       <mass
-        value="0" />
+        value="0.1" />
       <inertia
         ixx="0"

Commit message: Possibly rplidar works in autonomy_onboard.launch.py

File: ros2/description/urdf/ros2_control.xacro (robot description, xacro)
@@ -11,5 +11,5 @@
             </hardware>
             <!-- Define all the joints that will have a command or state interface -->
-            <joint name="DL_Rotate">
+            <joint name="Left Kraken">
                 <command_interface name="velocity">
                     <param name="min">-10</param>
@@ -19,5 +19,5 @@
                 <state_interface name="velocity"/>
             </joint>
-            <joint name="DR_Rotate">
+            <joint name="Left Kraken">
                 <command_interface name="velocity">
                     <param name="min">-10</param>
@@ -27,10 +27,10 @@
                 <state_interface name="velocity"/>
             </joint>
-            <joint name="LA_Extend">
+            <joint name="BLA Pivot">
                 <command_interface name="position"/>
                 <command_interface name="la_reset"/>
                 <state_interface name="position"/>
             </joint>
-            <joint name="Excavation_Rotate">
+            <joint name="E Roller">
                 <command_interface name="velocity">
                     <param name="min">-10</param>
