Commit message: replaced Back, middle, and front wheel collisions with spheres

File: ros2/description/urdf/tibble_core.xacro (robot description, xacro)
@@ -597,6 +597,7 @@
         rpy="0 0 0" />
       <geometry>
-        <mesh
-          filename="file://$(find description)/meshes/FL_Wheel.STL" />
+        <!-- <mesh
+          filename="file://$(find description)/meshes/FL_Wheel.STL" /> -->
+          <sphere radius="0.0929"/>
       </geometry>
     </collision>
@@ -650,6 +651,7 @@
         rpy="0 0 0" />
       <geometry>
-        <mesh
-          filename="file://$(find description)/meshes/ML_Wheel.STL" />
+        <!-- <mesh
+          filename="file://$(find description)/meshes/ML_Wheel.STL" /> -->
+          <sphere radius="0.0929"/>
       </geometry>
     </collision>
@@ -703,6 +705,7 @@
         rpy="0 0 0" />
       <geometry>
-        <mesh
-          filename="file://$(find description)/meshes/BL_Wheel.STL" />
+        <!-- <mesh
+          filename="file://$(find description)/meshes/BL_Wheel.STL" /> -->
+          <sphere radius="0.0929"/>
       </geometry>
     </collision>
@@ -809,6 +812,7 @@
         rpy="0 0 0" />
       <geometry>
-        <mesh
-          filename="file://$(find description)/meshes/FR_Wheel.STL" />
+        <!-- <mesh
+          filename="file://$(find description)/meshes/FR_Wheel.STL" /> -->
+          <sphere radius="0.0929"/>
       </geometry>
     </collision>
@@ -862,6 +866,7 @@
         rpy="0 0 0" />
       <geometry>
-        <mesh
-          filename="file://$(find description)/meshes/MR_Wheel.STL" />
+        <!-- <mesh
+          filename="file://$(find description)/meshes/MR_Wheel.STL" /> -->
+          <sphere radius="0.0929"/>
       </geometry>
     </collision>
@@ -915,6 +920,7 @@
         rpy="0 0 0" />
       <geometry>
-        <mesh
-          filename="file://$(find description)/meshes/BR_Wheel.STL" />
+        <!-- <mesh
+          filename="file://$(find description)/meshes/BR_Wheel.STL" /> -->
+          <sphere radius="0.0929"/>
       </geometry>
     </collision>

Commit message: did weird things to maybe make controller work

File: ros2/description/urdf/tibble_core.xacro (robot description, xacro)
@@ -218,4 +218,5 @@
       effort="0"
       velocity="0" />
+    <limit lower="0" upper="0.1" effort="100" velocity="1.0"/>
   </joint>
   <link
@@ -334,4 +335,5 @@
       effort="0"
       velocity="0" />
+    <limit lower="0" upper="0" effort="100" velocity="1.0"/>
   </joint>
   <link
@@ -670,4 +672,5 @@
     <axis
       xyz="0 0 -1" />
+    <dynamics damping="0.001" friction="0.0"/>
   </joint>
   <link
@@ -887,4 +890,5 @@
     <axis
       xyz="0 0 -1" />
+    <dynamics damping="0.001" friction="0.0"/>
   </joint>
   <link

Commit message: added new urdf in

File: ros2/description/urdf/tibble_core.xacro (robot description, xacro)
@@ -8,46 +8,46 @@
     <inertial>
       <origin
-        xyz="0.88193 1.2843 1.595"
-        rpy="0 0 0" />
-      <mass
-        value="5.3252" />
-      <inertia
-        ixx="0.016501"
-        ixy="-1.6464E-09"
-        ixz="0.0014196"
-        iyy="0.28053"
-        iyz="3.4252E-11"
-        izz="0.27372" />
-    </inertial>
-    <visual>
-      <origin
-        xyz="0 0 0"
-        rpy="0 0 0" />
-      <geometry>
-        <mesh
-          filename="file://$(find description)/meshes/Chassis.STL" />
-      </geometry>
-      <material
-        name="">
-        <color
-          rgba="0.25098 0.25098 0.25098 1" />
-      </material>
-    </visual>
-    <collision>
-      <origin
-        xyz="0 0 0"
-        rpy="0 0 0" />
-      <geometry>
-        <mesh
-          filename="file://$(find description)/meshes/Chassis.STL" />
-      </geometry>
-    </collision>
-  </link>
-    <joint
+        xyz="0.132671447387039 0.0508890561368854 -0.0113307002180522"
+        rpy="0 0 0" />
+      <mass
+        value="7.35143473795031" />
+      <inertia
+        ixx="0.213243148347066"
+        ixy="-0.00391416585919187"
+        ixz="5.52932059374091E-05"
+        iyy="0.037555624291398"
+        iyz="2.04129236166961E-06"
+        izz="0.203351368041528" />
+    </inertial>
+    <visual>
+      <origin
+        xyz="0 0 0"
+        rpy="0 0 0" />
+      <geometry>
+        <mesh
+          filename="file://$(find description)/meshes/chassis_link.STL" />
+      </geometry>
+      <material
+        name="">
+        <color
+          rgba="0.250980392156863 0.250980392156863 0.250980392156863 1" />
+      </material>
+    </visual>
+    <collision>
+      <origin
+        xyz="0 0 0"
+        rpy="0 0 0" />
+      <geometry>
+        <mesh
+          filename="file://$(find description)/meshes/chassis_link.STL" />
+      </geometry>
+    </collision>
+  </link>
+  <joint
     name="chassis"
     type="fixed">
     <origin
       xyz="0 0 0"
-      rpy="${-pi/2} 0 0" />
+      rpy="0 ${-pi/2} 0" />
     <parent
       link="base_link" />
@@ -56,79 +56,79 @@
   </joint>
   <link
-    name="DL_Wheel">
-    <inertial>
-      <origin
-        xyz="-2.6735E-11 -2.2271E-11 5.6577E-12"
-        rpy="0 0 0" />
-      <mass
-        value="0.17677" />
-      <inertia
-        ixx="0.00011937"
-        ixy="-6.5392E-14"
-        ixz="3.4896E-14"
-        iyy="0.00011937"
-        iyz="-1.0101E-14"
-        izz="0.00021546" />
-    </inertial>
-    <visual>
-      <origin
-        xyz="0 0 0"
-        rpy="0 0 0" />
-      <geometry>
-        <mesh
-          filename="file://$(find description)/meshes/DL_Wheel.STL" />
-      </geometry>
-      <material
-        name="">
-        <color
-          rgba="0.79216 0.81961 0.93333 1" />
-      </material>
-    </visual>
-    <collision>
-      <origin
-        xyz="0 0 0"
-        rpy="0 0 0" />
-      <geometry>
-        <mesh
-          filename="file://$(find description)/meshes/DL_Wheel.STL" />
-      </geometry>
-    </collision>
-  </link>
-  <joint
-    name="DL_Rotate"
+    name="DL_Continuous">
+    <inertial>
+      <origin
+        xyz="2.85323938087334E-10 -5.34546376292078E-06 -0.04591965264313"
+        rpy="0 0 0" />
+      <mass
+        value="0.276551696493172" />
+      <inertia
+        ixx="0.000210739473365903"
+        ixy="-4.91353538964495E-12"
+        ixz="2.72007860686062E-12"
+        iyy="0.000210739484819301"
+        iyz="1.6216820249958E-12"
+        izz="0.000304282368313418" />
+    </inertial>
+    <visual>
+      <origin
+        xyz="0 0 0"
+        rpy="0 0 0" />
+      <geometry>
+        <mesh
+          filename="file://$(find description)/meshes/DL_Continuous.STL" />
+      </geometry>
+      <material
+        name="">
+        <color
+          rgba="0.792156862745098 0.819607843137255 0.933333333333333 1" />
+      </material>
+    </visual>
+    <collision>
+      <origin
+        xyz="0 0 0"
+        rpy="0 0 0" />
+      <geometry>
+        <mesh
+          filename="file://$(find description)/meshes/DL_Continuous.STL" />
+      </geometry>
+    </collision>
+  </link>
+  <joint
+    name="Left Kraken"
     type="continuous">
     <origin
-      xyz="1.1775 -1.6339 1.5673"
-      rpy="3.1416 0 0.5236" />
-    <parent
-      link="chassis_link" />
-    <child
-      link="DL_Wheel" />
-    <axis
-      xyz="0 0 -1" />
-  </joint>
-  <link
-    name="DR_Wheel">
-    <inertial>
-      <origin
-        xyz="-2.67351696336959E-11 -2.22715179631905E-11 5.65791857809472E-12"
-        rpy="0 0 0" />
-      <mass
-        value="0.176769243894823" />
-      <inertia
-        ixx="0.000119374362744726"
-        ixy="-6.53920243420727E-14"
-        ixz="3.48950358018505E-14"
-        iyy="0.000119374363023012"
-        iyz="-1.01023471885648E-14"
-        izz="0.000215461530204446" />
-    </inertial>
-    <visual>
-      <origin
-        xyz="0 0 0"
-        rpy="0 0 0" />
-      <geometry>
-        <mesh
-          filename="file://$(find description)/meshes/DR_Wheel.STL" />
+      xyz="0.0635 0.32899 -0.030912"
+      rpy="-1.5708 -1.5705 0" />
+    <parent
+      link="chassis_link" />
+    <child
+      link="DL_Continuous" />
+    <axis
+      xyz="0 0 1" />
+  </joint>
+  <link
+    name="DR_Continuous">
+    <inertial>
+      <origin
+        xyz="4.01755715501162E-10 -5.34556506777417E-06 -0.0429803475776347"
+        rpy="0 0 0" />
+      <mass
+        value="0.27655169508797" />
+      <inertia
+        ixx="0.000210739474520998"
+        ixy="-7.07200276849857E-12"
+        ixz="2.74710832395788E-12"
+        iyy="0.000210739482055889"
+        iyz="1.60163314032096E-12"
+        izz="0.0003042823667301" />
+    </inertial>
+    <visual>
+      <origin
+        xyz="0 0 0"
+        rpy="0 0 0" />
+      <geometry>
+        <mesh
+          filename="file://$(find description)/meshes/DR_Continuous.STL" />
       </geometry>
       <material
@@ -144,44 +144,44 @@
       <geometry>
         <mesh
-          filename="file://$(find description)/meshes/DR_Wheel.STL" />
-      </geometry>
-    </collision>
-  </link>
-  <joint
-    name="DR_Rotate"
+          filename="file://$(find description)/meshes/DR_Continuous.STL" />
+      </geometry>
+    </collision>
+  </link>
+  <joint
+    name="Right Kraken"
     type="continuous">
     <origin
-      xyz="1.1775 -1.6339 1.0014"
-      rpy="3.1416 0 0.5236" />
-    <parent
-      link="chassis_link" />
-    <child
-      link="DR_Wheel" />
-    <axis
-      xyz="0 0 -1" />
-  </joint>
-  <link
-    name="BLA">
-    <inertial>
-      <origin
-        xyz="-0.0172681243630312 -0.116440645758096 0.212737229814056"
-        rpy="0 0 0" />
-      <mass
-        value="0.97023402841067" />
-      <inertia
-        ixx="0.00819569952353813"
-        ixy="0.000828153171744282"
-        ixz="-1.42662335730119E-06"
-        iyy="0.000699830914870433"
-        iyz="3.45710523187761E-06"
-        izz="0.00867844294735175" />
-    </inertial>
-    <visual>
-      <origin
-        xyz="0 0 0"
-        rpy="0 0 0" />
-      <geometry>
-        <mesh
-          filename="file://$(find description)/meshes/BLA.STL" />
+      xyz="0.0635 -0.24009 -0.030912"
+      rpy="-1.5708 -1.5705 0" />
+    <parent
+      link="chassis_link" />
+    <child
+      link="DR_Continuous" />
+    <axis
+      xyz="0 0 1" />
+  </joint>
+  <link
+    name="LA_Revolute">
+    <inertial>
+      <origin
+        xyz="-0.0172682421533344 -0.116440577073067 -3.35022004493087E-05"
+        rpy="0 0 0" />
+      <mass
+        value="0.970233115937581" />
+      <inertia
+        ixx="0.00819568975487689"
+        ixy="0.000828146435470868"
+        ixz="-1.42510665626676E-06"
+        iyy="0.000699827484011564"
+        iyz="3.45567010872927E-06"
+        izz="0.00867843043495149" />
+    </inertial>
+    <visual>
+      <origin
+        xyz="0 0 0"
+        rpy="0 0 0" />
+      <geometry>
+        <mesh
+          filename="file://$(find description)/meshes/LA_Revolute.STL" />
       </geometry>
       <material
@@ -197,49 +197,49 @@
       <geometry>
         <mesh
-          filename="file://$(find description)/meshes/BLA.STL" />
-      </geometry>
-    </collision>
-  </link>
-  <joint
-    name="LLA_Rotate"
+          filename="file://$(find description)/meshes/LA_Revolute.STL" />
+      </geometry>
+    </collision>
+  </link>
+  <joint
+    name="BLA Pivot"
     type="revolute">
     <origin
-      xyz="0.56252 -1.6364 1.0715"
-      rpy="0 0 0.88895" />
-    <parent
-      link="chassis_link" />
-    <child
-      link="BLA" />
+      xyz="0.066 0 0.58407"
+      rpy="1.5708 0.37611 -3.1416" />
+    <parent
+      link="chassis_link" />
+    <child
+      link="LA_Revolute" />
     <axis
       xyz="0 0 -1" />
     <limit
       lower="0"
-      upper="0.1"
-      effort="0"
+      upper="0.9"
+      effort="0.1"
       velocity="0" />
   </joint>
   <link
-    name="LA">
-    <inertial>
-      <origin
-        xyz="0.0420523159099391 0.0218514549059925 3.83189571184772E-08"
-        rpy="0 0 0" />
-      <mass
-        value="0.0898377249563414" />
-      <inertia
-        ixx="0.000634301272313686"
-        ixy="-3.23718441672287E-11"
-        ixz="-1.23742704912369E-10"
-        iyy="4.44119295047458E-06"
-        iyz="1.42114602862497E-10"
-        izz="0.000634330189167566" />
-    </inertial>
-    <visual>
-      <origin
-        xyz="0 0 0"
-        rpy="0 0 0" />
-      <geometry>
-        <mesh
-          filename="file://$(find description)/meshes/LA.STL" />
+    name="LA Pin Prismatic">
+    <inertial>
+      <origin
+        xyz="-9.94845673618627E-08 -0.229844966975777 0.201033022254761"
+        rpy="0 0 0" />
+      <mass
+        value="0.179675434898673" />
+      <inertia
+        ixx="0.00126860246345071"
+        ixy="-6.56099085456245E-11"
+        ixz="-2.47366456867446E-10"
+        iyy="8.88238541193122E-06"
+        iyz="2.82264180062203E-10"
+        izz="0.00126866030171068" />
+    </inertial>
+    <visual>
+      <origin
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
File: ros2/description/urdf/tibble_core_old.xacro (robot description, xacro)
@@ -44,5 +44,5 @@
     </collision>
   </link>
-  <joint
+    <joint
     name="chassis"
     type="fixed">
@@ -275,5 +275,5 @@
       upper="0.254"
       effort="2000"
-      velocity="0.006" /> <!-- upper: 10 inch stroke. effort: 250lbs max load into newtons. velocity: 6mm/s into m/s -->
+      velocity="0.006" />
   </joint>
   <link
@@ -389,5 +389,5 @@
     <limit
       lower="-1"
-      upper="1"
+      upper="0"
       effort="0"
       velocity="0" />
