Commit message: swapped file// uri to package// so it works in foxglove

File: ros2/description/urdf/tibble_core.xacro (robot description, xacro)
@@ -26,5 +26,5 @@
       <geometry>
         <mesh
-          filename="file://$(find description)/meshes/Chassis.STL" />
+          filename="package://description/meshes/Chassis.STL" />
       </geometry>
       <material
@@ -40,5 +40,5 @@
       <geometry>
         <mesh
-          filename="file://$(find description)/meshes/Chassis.STL" />
+          filename="package://description/meshes/Chassis.STL" />
       </geometry>
     </collision>
@@ -77,5 +77,5 @@
       <geometry>
         <mesh
-          filename="file://$(find description)/meshes/DL_Wheel.STL" />
+          filename="package://description/meshes/DL_Wheel.STL" />
       </geometry>
       <material
@@ -91,5 +91,5 @@
       <geometry>
         <mesh
-          filename="file://$(find description)/meshes/DL_Wheel.STL" />
+          filename="package://description/meshes/DL_Wheel.STL" />
       </geometry>
     </collision>
@@ -130,19 +130,19 @@
       <geometry>
         <mesh
-          filename="file://$(find description)/meshes/DR_Wheel.STL" />
-      </geometry>
-      <material
-        name="">
-        <color
-          rgba="0.792156862745098 0.819607843137255 0.933333333333333 1" />
-      </material>
-    </visual>
-    <collision>
-      <origin
-        xyz="0 0 0"
-        rpy="0 0 0" />
-      <geometry>
-        <mesh
-          filename="file://$(find description)/meshes/DR_Wheel.STL" />
+          filename="package://description/meshes/DR_Wheel.STL" />
+      </geometry>
+      <material
+        name="">
+        <color
+          rgba="0.792156862745098 0.819607843137255 0.933333333333333 1" />
+      </material>
+    </visual>
+    <collision>
+      <origin
+        xyz="0 0 0"
+        rpy="0 0 0" />
+      <geometry>
+        <mesh
+          filename="package://description/meshes/DR_Wheel.STL" />
       </geometry>
     </collision>
@@ -183,19 +183,19 @@
       <geometry>
         <mesh
-          filename="file://$(find description)/meshes/BLA.STL" />
-      </geometry>
-      <material
-        name="">
-        <color
-          rgba="0.792156862745098 0.819607843137255 0.933333333333333 1" />
-      </material>
-    </visual>
-    <collision>
-      <origin
-        xyz="0 0 0"
-        rpy="0 0 0" />
-      <geometry>
-        <mesh
-          filename="file://$(find description)/meshes/BLA.STL" />
+          filename="package://description/meshes/BLA.STL" />
+      </geometry>
+      <material
+        name="">
+        <color
+          rgba="0.792156862745098 0.819607843137255 0.933333333333333 1" />
+      </material>
+    </visual>
+    <collision>
+      <origin
+        xyz="0 0 0"
+        rpy="0 0 0" />
+      <geometry>
+        <mesh
+          filename="package://description/meshes/BLA.STL" />
       </geometry>
     </collision>
@@ -241,19 +241,19 @@
       <geometry>
         <mesh
-          filename="file://$(find description)/meshes/LA.STL" />
-      </geometry>
-      <material
-        name="">
-        <color
-          rgba="0.792156862745098 0.819607843137255 0.933333333333333 1" />
-      </material>
-    </visual>
-    <collision>
-      <origin
-        xyz="0 0 0"
-        rpy="0 0 0" />
-      <geometry>
-        <mesh
-          filename="file://$(find description)/meshes/LA.STL" />
+          filename="package://description/meshes/LA.STL" />
+      </geometry>
+      <material
+        name="">
+        <color
+          rgba="0.792156862745098 0.819607843137255 0.933333333333333 1" />
+      </material>
+    </visual>
+    <collision>
+      <origin
+        xyz="0 0 0"
+        rpy="0 0 0" />
+      <geometry>
+        <mesh
+          filename="package://description/meshes/LA.STL" />
       </geometry>
     </collision>
@@ -299,19 +299,19 @@
       <geometry>
         <mesh
-          filename="file://$(find description)/meshes/TLA.STL" />
-      </geometry>
-      <material
-        name="">
-        <color
-          rgba="0.792156862745098 0.819607843137255 0.933333333333333 1" />
-      </material>
-    </visual>
-    <collision>
-      <origin
-        xyz="0 0 0"
-        rpy="0 0 0" />
-      <geometry>
-        <mesh
-          filename="file://$(find description)/meshes/TLA.STL" />
+          filename="package://description/meshes/TLA.STL" />
+      </geometry>
+      <material
+        name="">
+        <color
+          rgba="0.792156862745098 0.819607843137255 0.933333333333333 1" />
+      </material>
+    </visual>
+    <collision>
+      <origin
+        xyz="0 0 0"
+        rpy="0 0 0" />
+      <geometry>
+        <mesh
+          filename="package://description/meshes/TLA.STL" />
       </geometry>
     </collision>
@@ -357,5 +357,5 @@
       <geometry>
         <mesh
-          filename="file://$(find description)/meshes/Hopper.STL" />
+          filename="package://description/meshes/Hopper.STL" />
       </geometry>
       <material
@@ -371,5 +371,5 @@
       <geometry>
         <mesh
-          filename="file://$(find description)/meshes/Hopper.STL" />
+          filename="package://description/meshes/Hopper.STL" />
       </geometry>
     </collision>
@@ -415,5 +415,5 @@
       <geometry>
         <mesh
-          filename="file://$(find description)/meshes/Hopper_Door.STL" />
+          filename="package://description/meshes/Hopper_Door.STL" />
       </geometry>
       <material
@@ -429,5 +429,5 @@
       <geometry>
         <mesh
-          filename="file://$(find description)/meshes/Hopper_Door.STL" />
+          filename="package://description/meshes/Hopper_Door.STL" />
       </geometry>
     </collision>
@@ -473,5 +473,5 @@
       <geometry>
         <mesh
-          filename="file://$(find description)/meshes/Hopper_Latch.STL" />
+          filename="package://description/meshes/Hopper_Latch.STL" />
       </geometry>
       <material
@@ -487,5 +487,5 @@
       <geometry>
         <mesh
-          filename="file://$(find description)/meshes/Hopper_Latch.STL" />
+          filename="package://description/meshes/Hopper_Latch.STL" />
       </geometry>
     </collision>
@@ -531,19 +531,19 @@
       <geometry>
         <mesh
-          filename="file://$(find description)/meshes/Excavation.STL" />
-      </geometry>
-      <material
-        name="">
-        <color
-          rgba="0.792156862745098 0.819607843137255 0.933333333333333 1" />
-      </material>
-    </visual>
-    <collision>
-      <origin
-        xyz="0 0 0"
-        rpy="0 0 0" />
-      <geometry>
-        <mesh
-          filename="file://$(find description)/meshes/Excavation.STL" />
+          filename="package://description/meshes/Excavation.STL" />
+      </geometry>
+      <material
+        name="">
+        <color
+          rgba="0.792156862745098 0.819607843137255 0.933333333333333 1" />
+      </material>
+    </visual>
+    <collision>
+      <origin
+        xyz="0 0 0"
+        rpy="0 0 0" />
+      <geometry>
+        <mesh
+          filename="package://description/meshes/Excavation.STL" />
       </geometry>
     </collision>
@@ -584,19 +584,19 @@
       <geometry>
         <mesh
-          filename="file://$(find description)/meshes/FL_Wheel.STL" />
-      </geometry>
-      <material
-        name="">
-        <color
-          rgba="0.792156862745098 0.819607843137255 0.933333333333333 1" />
-      </material>
-    </visual>
-    <collision>
-      <origin
-        xyz="0 0 0"
-        rpy="0 0 0" />
-      <geometry>
-        <mesh
-          filename="file://$(find description)/meshes/FL_Wheel.STL" />
+          filename="package://description/meshes/FL_Wheel.STL" />
+      </geometry>
+      <material
+        name="">
+        <color
+          rgba="0.792156862745098 0.819607843137255 0.933333333333333 1" />
+      </material>
+    </visual>
+    <collision>
+      <origin
+        xyz="0 0 0"
+        rpy="0 0 0" />
+      <geometry>
+        <mesh
+          filename="package://description/meshes/FL_Wheel.STL" />
       </geometry>
     </collision>
@@ -637,19 +637,19 @@
       <geometry>
         <mesh
-          filename="file://$(find description)/meshes/ML_Wheel.STL" />
-      </geometry>
-      <material
-        name="">
-        <color
-          rgba="0.792156862745098 0.819607843137255 0.933333333333333 1" />
-      </material>
-    </visual>
-    <collision>
-      <origin
-        xyz="0 0 0"
-        rpy="0 0 0" />
-      <geometry>
-        <mesh
-          filename="file://$(find description)/meshes/ML_Wheel.STL" />
+          filename="package://description/meshes/ML_Wheel.STL" />
+      </geometry>
+      <material
+        name="">
+        <color
+          rgba="0.792156862745098 0.819607843137255 0.933333333333333 1" />
+      </material>
+    </visual>
+    <collision>
+      <origin
+        xyz="0 0 0"
+        rpy="0 0 0" />
+      <geometry>
+        <mesh
+          filename="package://description/meshes/ML_Wheel.STL" />
       </geometry>
     </collision>
@@ -690,19 +690,19 @@
       <geometry>
         <mesh
-          filename="file://$(find description)/meshes/BL_Wheel.STL" />
-      </geometry>
-      <material
-        name="">
-        <color
-          rgba="0.792156862745098 0.819607843137255 0.933333333333333 1" />
-      </material>
-    </visual>
-    <collision>
-      <origin
-        xyz="0 0 0"
-        rpy="0 0 0" />
-      <geometry>
-        <mesh
-          filename="file://$(find description)/meshes/BL_Wheel.STL" />
+          filename="package://description/meshes/BL_Wheel.STL" />
+      </geometry>
+      <material
+        name="">
+        <color
+          rgba="0.792156862745098 0.819607843137255 0.933333333333333 1" />
+      </material>
+    </visual>
+    <collision>
+      <origin
+        xyz="0 0 0"
+        rpy="0 0 0" />
+      <geometry>
+        <mesh
+          filename="package://description/meshes/BL_Wheel.STL" />
       </geometry>
     </collision>
@@ -743,19 +743,19 @@
       <geometry>
         <mesh
-          filename="file://$(find description)/meshes/TL_Wheel.STL" />
-      </geometry>
-      <material
-        name="">
-        <color
-          rgba="0.792156862745098 0.819607843137255 0.933333333333333 1" />
-      </material>
-    </visual>
-    <collision>
-      <origin
-        xyz="0 0 0"
-        rpy="0 0 0" />
-      <geometry>
-        <mesh
-          filename="file://$(find description)/meshes/TL_Wheel.STL" />
+          filename="package://description/meshes/TL_Wheel.STL" />
+      </geometry>
+      <material
+        name="">
+        <color
+          rgba="0.792156862745098 0.819607843137255 0.933333333333333 1" />
+      </material>
+    </visual>
+    <collision>
+      <origin
+        xyz="0 0 0"
+        rpy="0 0 0" />
+      <geometry>
+        <mesh
+          filename="package://description/meshes/TL_Wheel.STL" />
       </geometry>
     </collision>
@@ -796,19 +796,19 @@
       <geometry>
         <mesh
-          filename="file://$(find description)/meshes/FR_Wheel.STL" />
-      </geometry>
-      <material
-        name="">
-        <color
-          rgba="0.792156862745098 0.819607843137255 0.933333333333333 1" />
-      </material>
-    </visual>
-    <collision>
-      <origin
-        xyz="0 0 0"
-        rpy="0 0 0" />
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
Commit message: Add urdf to mjcf converter in launch file

File: ros2/description/urdf/tibble_core.xacro (robot description, xacro)
@@ -937,15 +937,15 @@
     <inertial>
       <origin
-        xyz="0 0 0"
-        rpy="0 0 0" />
-      <mass
-        value="0" />
-      <inertia
-        ixx="0"
-        ixy="0"
-        ixz="0"
-        iyy="0"
-        iyz="0"
-        izz="0" />
+        xyz="-5.55111512312578E-17 0 -0.00138135898913294"
+        rpy="0 0 0" />
+      <mass
+        value="0.146434890659902" />
+      <inertia
+        ixx="8.80633224784676E-05"
+        ixy="-2.39106895777931E-22"
+        ixz="-1.34026306833892E-19"
+        iyy="8.80633224784676E-05"
+        iyz="-4.00087992203459E-19"
+        izz="0.000154471460357356" />
     </inertial>
     <visual>
